Commit message: [description] Add meshes + adapt URDF

File: ceol_description/urdf/ceol.urdf.xacro (robot description, xacro)
@@ -1,4 +1,4 @@
 <?xml version='1.0' encoding='utf-8'?>
-<robot name="aroco" xmlns:xacro="http://www.ros.org/wiki/xacro">
+<robot name="ceol" xmlns:xacro="http://www.ros.org/wiki/xacro">
   <xacro:arg name="prefix" default="ceol_" />
   <xacro:arg name="mode" default="simulation" />
@@ -6,7 +6,7 @@
   <xacro:arg name="ros2_control_config_urdf_file" default="" />
   <xacro:arg name="controller_manager_config_yaml_file" default="" />
-  <xacro:arg name="ros_prefix" default="/aroco/" />
+  <xacro:arg name="ros_prefix" default="/ceol/" />
   <xacro:include filename="$(find ceol_description)/urdf/ceol.xacro" />
-  <xacro:aroco mode="$(arg mode)" prefix="$(arg prefix)" />
+  <xacro:ceol mode="$(arg mode)" prefix="$(arg prefix)" />
   <gazebo>
     <plugin filename="libromea_gazebo_ros2_control.so" name="gazebo_ros2_control">

File: ceol_description/urdf/ceol.xacro (robot description, xacro)
@@ -1,4 +1,5 @@
 <?xml version="1.0"?>
-<robot name="aroco" xmlns:xacro="http://www.ros.org/wiki/xacro">
+<robot name="ceol" xmlns:xacro="http://www.ros.org/wiki/xacro">
+  <!-- <xacro:include filename="$(find ceol_description)/urdf/color.xacro" /> -->
   <xacro:include filename="$(find romea_mobile_base_description)/urdf/base2THD.chassis.xacro" />
   <xacro:property name="conf" value="$(find ceol_description)/config/ceol.yaml" />
@@ -80,24 +81,25 @@
   <xacro:property name="chassis_height"
     value="${props['geometry']['tracks']['front_idler_wheel']['radius']}" />
-  <xacro:macro name="aroco" params="mode prefix">
+  <xacro:macro name="ceol" params="mode prefix">
     <!-- visual chassis -->
     <xacro:chassis>
       <!-- visual chassis -->
+      <!-- <visual> -->
+      <!--   <geometry> -->
+      <!--     <box size="${aabb_length} ${aabb_width} ${aabb_height}"/> -->
+      <!--   </geometry> -->
+      <!--   <origin xyz="${aabb_center_x-body_reference_x} ${aabb_center_y}  ${aabb_center_z-chassis_height}" rpy="0 0 0" /> -->
+      <!--   <material name="grey"> -->
+      <!--     &#60;&#33;&#45;&#45; <color rgba="0.6 0.6 0.6 1"/> &#45;&#45;&#62; -->
+      <!--     <color rgba="0.99 0.6 0.6 1"/> -->
+      <!--   </material> -->
+      <!-- </visual> -->
       <visual>
+        <origin xyz="0 0 0" rpy="0 0 ${pi/2}" />
         <geometry>
-          <box size="${aabb_length} ${aabb_width} ${aabb_height}"/>
+          <!-- <box size="${aabb_length} ${aabb_width} ${aabb_height}"/> -->
+          <mesh filename="package://ceol_description/meshes/ceol.dae" />
         </geometry>
-        <origin xyz="${aabb_center_x-body_reference_x} ${aabb_center_y}  ${aabb_center_z-chassis_height}" rpy="0 0 0" />
-        <material name="grey">
-          <color rgba="0.6 0.6 0.6 1"/>
-        </material>
       </visual>
-      <!-- <visual>
-        <origin xyz="${0.03-body_reference_x} 0 ${chassis_height-aabb_height/2}"
-          rpy="0 0 ${M_PI/2.0}" />
-        <geometry>
-          <mesh filename="package://ceol_description/meshes/chassis.dae" />
-        </geometry>
-      </visual> -->
       <!-- visual sprocker wheel -->
       <cylinder length="${track_width}" radius="${sprocket_wheel_radius+track_thickness}"/>
@@ -107,4 +109,12 @@
       <!-- <mesh filename="package://ceol_description/meshes/idler_wheel.dae" /> -->
     </xacro:chassis>
+    <gazebo reference="${prefix}${base_link}">
+      <material>
+        <script>
+          <uri>package://alpo_description/meshes/ceol.material</uri>
+          <name>ceol</name>
+        </script>
+      </material>
+    </gazebo>
   </xacro:macro>
 </robot>
