Commit message: [description] separate wheel meshes to chassis

File: ceol_description/urdf/ceol.xacro (robot description, xacro)
@@ -99,5 +99,5 @@
         <geometry>
           <!-- <box size="${aabb_length} ${aabb_width} ${aabb_height}"/> -->
-          <mesh filename="package://ceol_description/meshes/ceol.dae" />
+          <mesh filename="package://ceol_description/meshes/ceol_chassis.dae" />
         </geometry>
       </visual>
@@ -109,4 +109,30 @@
       <!-- <mesh filename="package://ceol_description/meshes/idler_wheel.dae" /> -->
     </xacro:chassis>
+    <link name="${prefix}left_wheel_model">
+      <visual>
+        <origin xyz="0 0 0" rpy="0 0 ${pi/2}" />
+        <geometry>
+          <mesh filename="package://ceol_description/meshes/ceol_roue.dae" />
+        </geometry>
+      </visual>
+    </link>
+    <joint name="${prefix}left_wheel_model_joint" type="fixed">
+      <origin xyz="0 ${track/2} 0" rpy="0 0 0" />
+      <child link="${prefix}left_wheel_model" />
+      <parent link="${prefix}${base_link}" />
+    </joint>
+    <link name="${prefix}right_wheel_model">
+      <visual>
+        <origin xyz="0 0 0" rpy="0 0 ${pi/2}" />
+        <geometry>
+          <mesh filename="package://ceol_description/meshes/ceol_roue.dae" scale="-1 1 1"/>
+        </geometry>
+      </visual>
+    </link>
+    <joint name="${prefix}right_wheel_model_joint" type="fixed">
+      <origin xyz="0 ${-track/2} 0" rpy="0 0 0" />
+      <child link="${prefix}right_wheel_model" />
+      <parent link="${prefix}${base_link}" />
+    </joint>
     <gazebo reference="${prefix}${base_link}">
       <material>

Commit message: [description] rename ceol_roue to ceol_wheel

File: ceol_description/urdf/ceol.xacro (robot description, xacro)
@@ -113,5 +113,5 @@
         <origin xyz="0 0 0" rpy="0 0 ${pi/2}" />
         <geometry>
-          <mesh filename="package://ceol_description/meshes/ceol_roue.dae" />
+          <mesh filename="package://ceol_description/meshes/ceol_wheel.dae" />
         </geometry>
       </visual>
@@ -126,5 +126,5 @@
         <origin xyz="0 0 0" rpy="0 0 ${pi/2}" />
         <geometry>
-          <mesh filename="package://ceol_description/meshes/ceol_roue.dae" scale="-1 1 1"/>
+          <mesh filename="package://ceol_description/meshes/ceol_wheel.dae" scale="-1 1 1"/>
         </geometry>
       </visual>

Commit message: description: change way to add visuals in xacro file
Signed-off-by: jean.laneurit <jean.laneurit@inrae.fr>

File: ceol_description/urdf/ceol.xacro (robot description, xacro)
@@ -3,4 +3,6 @@
   <!-- <xacro:include filename="$(find ceol_description)/urdf/color.xacro" /> -->
   <xacro:include filename="$(find romea_mobile_base_description)/urdf/base2THD.chassis.xacro" />
+  <xacro:include filename="$(find ceol_description)/urdf/visual/chassis.xacro" />
+  <xacro:include filename="$(find ceol_description)/urdf/visual/wheels.xacro" />
   <xacro:property name="conf" value="$(find ceol_description)/config/ceol.yaml" />
   <xacro:property name="props" value="${load_yaml(conf)}" />
@@ -45,7 +47,7 @@
   <xacro:property name="aabb_center_z" value="${props['geometry']['aabb']['center'][2]}" />
   <xacro:property name="front_idler_wheel_x"
-    value= "${props['geometry']['tracks']['front_idler_wheel']['x']}"/>
+    value="${props['geometry']['tracks']['front_idler_wheel']['x']}" />
   <xacro:property name="rear_idler_wheel_x"
-    value= "${props['geometry']['tracks']['rear_idler_wheel']['x']}"/>
+    value="${props['geometry']['tracks']['rear_idler_wheel']['x']}" />
   <xacro:property name="wheelbase" value="${front_idler_wheel_x-rear_idler_wheel_x}" />
   <xacro:property name="track" value="${props['geometry']['tracks_distance']}" />
@@ -56,5 +58,5 @@
   <xacro:property name="mass_center_y" value="${props['inertia']['center'][1]}" />
   <xacro:property name="mass_center_z" value="${props['inertia']['center'][2]}" />
-   <xacro:property name="maximal_wheel_speed"
+  <xacro:property name="maximal_wheel_speed"
     value="${props['tracks_speed_control']['command']['maximal_speed']}" />
   <xacro:property name="body_reference_x" value="${props['control_point'][0]}" />
@@ -82,30 +84,10 @@
     value="${props['geometry']['tracks']['front_idler_wheel']['radius']}" />
   <xacro:macro name="ceol" params="mode prefix">
-    <!-- visual chassis -->
     <xacro:chassis>
-      <!-- visual chassis -->
-      <!-- <visual> -->
-      <!--   <geometry> -->
-      <!--     <box size="${aabb_length} ${aabb_width} ${aabb_height}"/> -->
-      <!--   </geometry> -->
-      <!--   <origin xyz="${aabb_center_x-body_reference_x} ${aabb_center_y}  ${aabb_center_z-chassis_height}" rpy="0 0 0" /> -->
-      <!--   <material name="grey"> -->
-      <!--     &#60;&#33;&#45;&#45; <color rgba="0.6 0.6 0.6 1"/> &#45;&#45;&#62; -->
-      <!--     <color rgba="0.99 0.6 0.6 1"/> -->
-      <!--   </material> -->
-      <!-- </visual> -->
-      <visual>
-        <origin xyz="0 0 0" rpy="0 0 ${pi/2}" />
-        <geometry>
-          <!-- <box size="${aabb_length} ${aabb_width} ${aabb_height}"/> -->
-          <mesh filename="package://ceol_description/meshes/ceol_chassis.dae" />
-        </geometry>
-      </visual>
-      <!-- visual sprocker wheel -->
-      <cylinder length="${track_width}" radius="${sprocket_wheel_radius+track_thickness}"/>
-      <!-- <mesh filename="package://ceol_description/meshes/sprocket_wheel.dae" /> -->
-      <!-- visual visual idler wheel -->
-      <cylinder length="${track_width}" radius="${idler_wheel_radius+track_thickness}"/>
-      <!-- <mesh filename="package://ceol_description/meshes/idler_wheel.dae" /> -->
+      <xacro:chassis_visual />
+      <xacro:left_sprocket_wheel_visual />
+      <xacro:right_sprocket_wheel_visual />
+      <xacro:left_idler_wheel_visual />
+      <xacro:right_idler_wheel_visual />
     </xacro:chassis>
     <link name="${prefix}left_wheel_model">
@@ -126,5 +108,5 @@
         <origin xyz="0 0 0" rpy="0 0 ${pi/2}" />
         <geometry>
-          <mesh filename="package://ceol_description/meshes/ceol_wheel.dae" scale="-1 1 1"/>
+          <mesh filename="package://ceol_description/meshes/ceol_wheel.dae" scale="-1 1 1" />
         </geometry>
       </visual>
@@ -138,9 +120,11 @@
       <material>
         <script>
-          <uri>package://alpo_description/meshes/ceol.material</uri>
+          <uri>package://ceol_description/meshes/ceol.material</uri>
           <name>ceol</name>
         </script>
       </material>
     </gazebo>
+    <!-- <xacro:include filename="$(find ceol_description)/urdf/three_hitch_point_ceol.urdf.xacro"
+    /> -->
   </xacro:macro>
 </robot>

Commit message: refactoring
Signed-off-by: Jean Laneurit <jean.laneurit@inrae.fr>

File: ceol_description/urdf/ceol.xacro (robot description, xacro)
@@ -95,5 +95,6 @@
         <origin xyz="0 0 0" rpy="0 0 ${pi/2}" />
         <geometry>
-          <mesh filename="package://ceol_description/meshes/ceol_wheel.dae" />
+          <!-- <mesh filename="package://ceol_description/meshes/ceol_wheel.dae" /> -->
+          <mesh filename="file://$(find ceol_description)/meshes/ceol_wheel.dae" />
         </geometry>
       </visual>
@@ -108,5 +109,6 @@
         <origin xyz="0 0 0" rpy="0 0 ${pi/2}" />
         <geometry>
-          <mesh filename="package://ceol_description/meshes/ceol_wheel.dae" scale="-1 1 1" />
+          <!-- <mesh filename="package://ceol_description/meshes/ceol_wheel.dae" scale="-1 1 1" /> -->
+          <mesh filename="file://$(find ceol_description)/meshes/ceol_wheel.dae" />
         </geometry>
       </visual>

File: ceol_description/urdf/visual/chassis.xacro (robot description, xacro)
@@ -6,5 +6,6 @@
             <geometry>
                 <!-- <box size="${aabb_length} ${aabb_width} ${aabb_height}"/> -->
-                <mesh filename="package://ceol_description/meshes/ceol_chassis.dae" />
+                <!-- <mesh filename="package://ceol_description/meshes/ceol_chassis.dae" /> -->
+                <mesh filename="file://$(find ceol_description)/meshes/ceol_chassis.dae" />
             </geometry>
         </visual>
