Commit message: add support of multi simulator
Signed-off-by: jean.laneurit <jean.laneurit@inrae.fr>

File: ceol_description/ros2_control/ceol.ros2_control.xacro (robot description, xacro)
@@ -29,6 +29,16 @@
       value="${props['tracks_speed_control']['command']['maximal_speed']}" />
     <!-- simulation plugins -->
-    <xacro:property name="simulation_hardware_plugin"
-      value="romea_mobile_base_gazebo/GazeboSystemInterface2THD" />
+    <xacro:if value="${'simulation' in mode}">
+      <xacro:if value="${'gazebo' in  mode}">
+        <xacro:property
+          name="simulation_hardware_plugin"
+          value="romea_mobile_base_gazebo/GazeboSystemInterface2THD" />
+      </xacro:if>
+      <xacro:if value="${'4dv' in  mode or 'isaac' in mode}">
+        <xacro:property
+          name="simulation_hardware_plugin"
+          value="romea_mobile_base_hardware/GenericHardwareSystemInterface2THD" />
+      </xacro:if>
+    </xacro:if>
     <xacro:property name="live_hardware_plugin"
       value="ceol_hardware/CeolHardware" />
