Commit message: [description] update xacro description files
Signed-off-by: Jean Laneurit <jean.laneurit@inrae.fr>

File: ceol_description/ros2_control/ceol.ros2_control.xacro (robot description, xacro)
@@ -28,20 +28,32 @@
     <xacro:property name="maximal_wheel_speed"
       value="${props['tracks_speed_control']['command']['maximal_speed']}" />
-    <!-- simulation plugins -->
-    <xacro:if value="${'simulation' in mode}">
-      <xacro:if value="${'gazebo' in  mode}">
-        <xacro:property
-          name="simulation_hardware_plugin"
-          value="romea_mobile_base_gazebo/GazeboSystemInterface2THD" />
-      </xacro:if>
-      <xacro:if value="${'4dv' in  mode or 'isaac' in mode}">
-        <xacro:property
-          name="simulation_hardware_plugin"
-          value="romea_mobile_base_hardware/GenericHardwareSystemInterface2THD" />
-      </xacro:if>
+    <!-- simulation control -->
+    <xacro:if value="${'simulation_gazebo' in mode}">
+      <xacro:simulation_base_control
+        mode="${mode}"
+        base_name="${base_name}"/>
     </xacro:if>
-    <xacro:property name="live_hardware_plugin"
-      value="ceol_hardware/CeolHardware" />
-    <xacro:base_control mode="${mode}" base_name="${base_name}" />
+    <xacro:if value="${mode == 'simulation_gazebo_classic'}">
+      <xacro:base_control
+        mode="${mode}"
+        base_name="${base_name}"
+        hardware_plugin="romea_mobile_base_gazebo/GazeboSystemInterface4WS4WD" />
+    </xacro:if>
+    <xacro:if value="${'4dv' in mode or 'isaac' in mode}">
+      <xacro:base_control
+        mode="${mode}"
+        base_name="${base_name}"
+        hardware_plugin="romea_mobile_base_simulation/GenericSimulationSystemInterface" />
+    </xacro:if>
+    <!-- live control -->
+    <xacro:if value="${mode =='live'}">
+      <ros2_control name="${prefix}${base_name}" type="system">
+        <hardware>
+          <plugin>ceol_hardware/CeolHardware</plugin>
+          <xacro:base_control_parameters/>
+        </hardware>
+        <xacro:base_control_joints mode="${mode}"/>
+      </ros2_control>
+    </xacro:if>
   </xacro:macro>
 </robot>

File: ceol_description/urdf/ceol.simulation.xacro (robot description, xacro)
@@ -18,16 +18,9 @@
       </xacro:if>
       <xacro:if value="${'gazebo_classic' not in  mode}">
-        <gazebo>
-          <plugin filename="gz_ros2_control-system"
-            name="gz_ros2_control::GazeboSimROS2ControlPlugin">
-            <robot_param>robot_description</robot_param>
-            <robot_param_node>ros2_control_description</robot_param_node>
-            <parameters>${controller_manager_config_yaml_file}</parameters>
-            <!-- <hold_joints>true</hold_joints> -->
-            <ros>
-              <namespace>${ros_prefix}${base_name}</namespace>
-            </ros>
-          </plugin>
-        </gazebo>
+        <xacro:ros2_control_gazebo_plugin
+          plugin_filename="gz_ros2_control-system"
+          plugin_name="gz_ros2_control::GazeboSimROS2ControlPlugin"
+          ros_namespace="${ros_prefix}${base_name}"
+          controller_manager_config_yaml_file="${controller_manager_config_yaml_file}"/>
       </xacro:if>
     </xacro:if>

File: ceol_description/urdf/ceol.urdf.xacro (robot description, xacro)
@@ -9,9 +9,12 @@
   <xacro:include filename="$(find ceol_description)/urdf/ceol.xacro" />
   <xacro:ceol mode="$(arg mode)" prefix="$(arg prefix)" />
-  <xacro:include filename="$(find ceol_description)/urdf/ceol.simulation.xacro" />
-  <xacro:ceol_simulation
-    mode="$(arg mode)"
-    base_name="$(arg base_name)"
-    ros_prefix="$(arg ros_prefix)"
-    controller_manager_config_yaml_file="$(arg controller_manager_config_yaml_file)" />
+  <xacro:if value="${'gazebo' in '$(arg mode)'}">
+    <xacro:include
+      filename="$(find romea_mobile_base_description)/urdf/gazebo_ros2_control.xacro" />
+    <xacro:gazebo_ros2_control
+      mode="$(arg mode)"
+      base_name="$(arg base_name)"
+      ros_prefix="$(arg ros_prefix)"
+      controller_manager_config_yaml_file="$(arg controller_manager_config_yaml_file)" />
+  </xacro:if>
 </robot>

Commit message: [description] add base properties.xacro + update base launch file to avoid duplicate joints in ros2_control urdf file
Signed-off-by: Jean Laneurit <jean.laneurit@inrae.fr>

File: ceol_description/ros2_control/ceol.ros2_control.xacro (robot description, xacro)
@@ -2,31 +2,6 @@
 <robot name="ceol" xmlns:xacro="http://www.ros.org/wiki/xacro">
   <xacro:macro name="ceol_ros2_control" params="mode prefix base_name">
-    <xacro:include
-      filename="$(find romea_mobile_base_description)/ros2_control/base2THD.ros2_control.xacro" />
-    <xacro:property name="conf" value="$(find ceol_description)/config/ceol.yaml" />
-    <xacro:property name="props" value="${load_yaml(conf)}" />
-    <!-- Joint names -->
-    <xacro:property name="left_sprocket_wheel_spinning_joint"
-      value="${props['joints']['left_sprocket_wheel_spinning_joint_name']}" />
-    <xacro:property name="right_sprocket_wheel_spinning_joint"
-      value="${props['joints']['right_sprocket_wheel_spinning_joint_name']}" />
-    <xacro:property name="front_left_idler_wheel_spinning_joint"
-      value="${props['joints']['front_left_idler_wheel_spinning_joint_name']}" />
-    <xacro:property name="front_right_idler_wheel_spinning_joint"
-      value="${props['joints']['front_right_idler_wheel_spinning_joint_name']}" />
-    <xacro:property name="rear_left_idler_wheel_spinning_joint"
-      value="${props['joints']['rear_left_idler_wheel_spinning_joint_name']}" />
-    <xacro:property name="rear_right_idler_wheel_spinning_joint"
-      value="${props['joints']['rear_right_idler_wheel_spinning_joint_name']}" />
-    <!-- Geometry -->
-    <xacro:property name="sprocket_wheel_radius"
-      value="${props['geometry']['tracks']['sprocket_wheel']['radius']}" />
-    <xacro:property name="idler_wheel_radius"
-      value="${props['geometry']['tracks']['front_idler_wheel']['radius']}" />
-    <xacro:property name="track_thickness"
-      value="${props['geometry']['tracks']['thickness']}" />
-    <xacro:property name="maximal_wheel_speed"
-      value="${props['tracks_speed_control']['command']['maximal_speed']}" />
-    <!-- simulation control -->
+    <xacro:include filename="$(find romea_mobile_base_description)/ros2_control/base2THD.ros2_control.xacro" />
+    <xacro:include filename="$(find ceol_description)/urdf/ceol_base_properties.xacro" />
     <xacro:if value="${'simulation_gazebo' == mode}">
       <xacro:simulation_base_control

File: ceol_description/urdf/ceol.xacro (robot description, xacro)
@@ -5,82 +5,5 @@
   <xacro:include filename="$(find ceol_description)/urdf/visual/chassis.xacro" />
   <xacro:include filename="$(find ceol_description)/urdf/visual/wheels.xacro" />
-  <xacro:property name="conf" value="$(find ceol_description)/config/ceol.yaml" />
-  <xacro:property name="props" value="${load_yaml(conf)}" />
-  <!-- Link names -->
-  <xacro:property name="base_link" value="${props['links']['base_link_name']}" />
-  <xacro:property name="base_footprint_link" value="${props['links']['base_footprint_link_name']}" />
-  <xacro:property name="inertial_link" value="${props['links']['inertial_link_name']}" />
-  <xacro:property name="left_sprocket_wheel_spinning_link"
-    value="${props['links']['left_sprocket_wheel_spinning_link_name']}" />
-  <xacro:property name="right_sprocket_wheel_spinning_link"
-    value="${props['links']['right_sprocket_wheel_spinning_link_name']}" />
-  <xacro:property name="front_left_idler_wheel_spinning_link"
-    value="${props['links']['front_left_idler_wheel_spinning_link_name']}" />
-  <xacro:property name="front_right_idler_wheel_spinning_link"
-    value="${props['links']['front_right_idler_wheel_spinning_link_name']}" />
-  <xacro:property name="rear_left_idler_wheel_spinning_link"
-    value="${props['links']['rear_left_idler_wheel_spinning_link_name']}" />
-  <xacro:property name="rear_right_idler_wheel_spinning_link"
-    value="${props['links']['rear_right_idler_wheel_spinning_link_name']}" />
-  <!-- Joint names -->
-  <xacro:property name="base_footprint_joint"
-    value="${props['joints']['base_footprint_joint_name']}" />
-  <xacro:property name="inertial_joint" value="${props['joints']['inertial_joint_name']}" />
-  <xacro:property name="left_sprocket_wheel_spinning_joint"
-    value="${props['joints']['left_sprocket_wheel_spinning_joint_name']}" />
-  <xacro:property name="right_sprocket_wheel_spinning_joint"
-    value="${props['joints']['right_sprocket_wheel_spinning_joint_name']}" />
-  <xacro:property name="front_left_idler_wheel_spinning_joint"
-    value="${props['joints']['front_left_idler_wheel_spinning_joint_name']}" />
-  <xacro:property name="front_right_idler_wheel_spinning_joint"
-    value="${props['joints']['front_right_idler_wheel_spinning_joint_name']}" />
-  <xacro:property name="rear_left_idler_wheel_spinning_joint"
-    value="${props['joints']['rear_left_idler_wheel_spinning_joint_name']}" />
-  <xacro:property name="rear_right_idler_wheel_spinning_joint"
-    value="${props['joints']['rear_right_idler_wheel_spinning_joint_name']}" />
-  <!-- Base Properties -->
-  <xacro:property name="aabb_length" value="${props['geometry']['aabb']['length']}" />
-  <xacro:property name="aabb_width" value="${props['geometry']['aabb']['width']}" />
-  <xacro:property name="aabb_height" value="${props['geometry']['aabb']['height']}" />
-  <xacro:property name="aabb_center_x" value="${props['geometry']['aabb']['center'][0]}" />
-  <xacro:property name="aabb_center_y" value="${props['geometry']['aabb']['center'][1]}" />
-  <xacro:property name="aabb_center_z" value="${props['geometry']['aabb']['center'][2]}" />
-  <xacro:property name="front_idler_wheel_x"
-    value="${props['geometry']['tracks']['front_idler_wheel']['x']}" />
-  <xacro:property name="rear_idler_wheel_x"
-    value="${props['geometry']['tracks']['rear_idler_wheel']['x']}" />
-  <xacro:property name="wheelbase" value="${front_idler_wheel_x-rear_idler_wheel_x}" />
-  <xacro:property name="track" value="${props['geometry']['tracks_distance']}" />
-  <xacro:property name="track_width" value="${props['geometry']['tracks']['width']}" />
-  <xacro:property name="track_thickness" value="${props['geometry']['tracks']['thickness']}" />
-  <xacro:property name="mass_base" value="${props['inertia']['mass']}" />
-  <xacro:property name="mass_center_x" value="${props['inertia']['center'][0]}" />
-  <xacro:property name="mass_center_y" value="${props['inertia']['center'][1]}" />
-  <xacro:property name="mass_center_z" value="${props['inertia']['center'][2]}" />
-  <xacro:property name="maximal_wheel_speed"
-    value="${props['tracks_speed_control']['command']['maximal_speed']}" />
-  <xacro:property name="body_reference_x" value="${props['control_point'][0]}" />
-  <!-- Wheel Properties -->
-  <xacro:property name="idler_wheel_mass"
-    value="${props['geometry']['tracks']['front_idler_wheel']['mass']}" />
-  <xacro:property name="idler_wheel_radius"
-    value="${props['geometry']['tracks']['front_idler_wheel']['radius']}" />
-  <xacro:property name="roller_wheel_mass"
-    value="${props['geometry']['tracks']['roller_wheels']['mass']}" />
-  <xacro:property name="roller_wheel_radius"
-    value="${props['geometry']['tracks']['roller_wheels']['radius']}" />
-  <xacro:property name="sprocket_wheel_mass"
-    value="${props['geometry']['tracks']['sprocket_wheel']['mass']}" />
-  <xacro:property name="sprocket_wheel_radius"
-    value="${props['geometry']['tracks']['sprocket_wheel']['radius']}" />
-  <xacro:property name="sprocket_wheel_x"
-    value="${props['geometry']['tracks']['sprocket_wheel']['x']}" />
-  <xacro:property name="sprocket_wheel_z"
-    value="${props['geometry']['tracks']['sprocket_wheel']['z']}" />
-  <!-- Wheel Mounting Positions -->
-  <xacro:property name="ground_clearance"
-    value="${props['geometry']['ground_clearance']}" />
-  <xacro:property name="chassis_height"
-    value="${props['geometry']['tracks']['front_idler_wheel']['radius']}" />
+  <xacro:include filename="$(find ceol_description)/urdf/ceol_base_properties.xacro" />
   <xacro:macro name="ceol" params="mode prefix">
     <xacro:chassis>
